File: east-van/east-van.kicad_pcb (KiCad board)
At the start: 2 copper layers, 49.4 x 83.3 mm, 10 parts

Commit message: East Van pcb as submitted
Parts:
- added H3: copper, east-van:east-van-copper, F.Cu at (110.1, 84.5)
- H1: value mech-only-no-pins -> mask; footprint east-van:east-van-mask -> east-van:east-van-inv-mask
- H2: value mech-only-no-pins -> silk
