File: deutsche-bahn/deutsche-bahn-sao.kicad_pcb (KiCad board)
At the start: 2 copper layers, 65 x 45.5 mm, 3 parts

Commit message: deutsche-bahn: v1.0 as submitted
Parts:
- removed G***: LOGO, deutsche-bahn-sao:1280px-Deutsche_Bahn_AG-Logo-silk-invert
- removed G***: LOGO, deutsche-bahn-sao:1280px-Deutsche_Bahn_AG-Logo-copper
- removed G***: LOGO, deutsche-bahn-sao:1280px-Deutsche_Bahn_AG-Logo-mask-invert
- added D1: LED, tom-opto:XZM2CYK45WT-9-NOMASK, B.Cu at (130.9, 79.9)
- added D10: LED, tom-opto:XZM2CYK45WT-9-NOMASK, B.Cu at (145.7, 89.5)
- added D11: LED, tom-opto:XZM2CYK45WT-9-NOMASK, B.Cu at (137.2, 74.0)
- added D12: LED, tom-opto:XZM2CYK45WT-9-NOMASK, B.Cu at (157.2, 92.7)
- added D13: LED, tom-opto:XZM2CYK45WT-9-NOMASK, B.Cu at (163.1, 99.1)
- added D2: LED, tom-opto:XZM2CYK45WT-9-NOMASK, B.Cu at (137.2, 99.1)
- added D3: LED, tom-opto:XZM2CYK45WT-9-NOMASK, B.Cu at (163.1, 73.9)
- added D4: LED, tom-opto:XZM2CYK45WT-9-NOMASK, B.Cu at (130.9, 89.9)
- added D5: LED, tom-opto:XZM2CYK45WT-9-NOMASK, B.Cu at (171.2, 78.9)
- added D6: LED, tom-opto:XZM2CYK45WT-9-NOMASK, B.Cu at (157.2, 79.9)
- added D7: LED, tom-opto:XZM2CYK45WT-9-NOMASK, B.Cu at (145.7, 80.5)
- added D8: LED, tom-opto:XZM2CYK45WT-9-NOMASK, B.Cu at (163.1, 85.9)
- added D9: LED, tom-opto:XZM2CYK45WT-9-NOMASK, B.Cu at (171.3, 92.7)
- added H1: Logo Copper, deutsche-bahn-sao:1280px-Deutsche_Bahn_AG-Logo-copper, F.Cu at (151.0, 86.4)
- added H2: Logo Mask, deutsche-bahn-sao:1280px-Deutsche_Bahn_AG-Logo-mask-invert, F.Cu at (151.0, 86.3)
- added H3: Logo Silk, deutsche-bahn-sao:1280px-Deutsche_Bahn_AG-Logo-silk-invert, F.Cu at (151.0, 86.3)
- added J1: Conn_02x03_Odd_Even, tom-connectors:PinSocket_2x03_P2.54mm_Vertical_SMD_SAO, B.Cu at (151.1, 109.2)
- added R1: 47R, tom-passives:C_0805_2012Metric_Pad1.15x1.40mm_HandSolder, B.Cu at (143.9, 98.2)
- added R2: 47R, tom-passives:C_0805_2012Metric_Pad1.15x1.40mm_HandSolder, B.Cu at (157.0, 98.2)
Routing:
- net +3V3: track 0.00 -> 190.7 mm
- net Net-(D1-Pad1): track 0.00 -> 84.8 mm
- net Net-(D12-Pad1): track 0.00 -> 62.3 mm
- net GND: track 0.00 -> 44.4 mm
Other:
- board size 65 x 45.5 mm -> 65 x 50.6 mm
- board text added: "db.tomk.in v1.0"
