File: east-van/arrow/east-van-arrow.kicad_pcb (KiCad board)
At the start: 2 copper layers, 29.2 x 64.9 mm, 10 parts, among them J1 Conn_02x03_Odd_Even

Commit message: east-van-arrow: v1.0 revised larger
Parts:
- moved D2 95.4 mm to (32.9, 61.0), turned to 0 degrees
- moved D1 93.8 mm to (44.0, 90.8), turned to 90 degrees
- moved D4 92.3 mm to (44.9, 42.6), turned to 8 degrees
- moved R1 86.7 mm to (34.8, 102.5)
- moved H2 85.5 mm to (45.0, 66.1)
- moved H1 85.5 mm to (45.0, 66.1)
- moved D3 83.6 mm to (44.0, 76.2), turned to 330 degrees
- moved J1 83.4 mm to (43.6, 108.6)
- moved D6 78.5 mm to (57.2, 58.7), turned to 300 degrees
- moved D5 76.8 mm to (44.0, 62.3), turned to 7 degrees
Routing:
- net /CATHODE: track 69.4 -> 154.9 mm
- net +3V3: track 107.1 -> 160.4 mm
- net GND: track 12.5 -> 10.1 mm
Other:
- board size 29.2 x 64.9 mm -> 44.9 x 88 mm
- board text added: "tom@tomk.in v1.0"

Commit message: eat-van-arrow: v1.1 fix issues with back solder mask
Other:
- board text added: "tom@tomk.in v1.1"
- board text removed: "tom@tomk.in v1.0"
Changed lines of the file:
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@@
-(kicad_pcb (version 20171130) (host pcbnew 5.1.4+dfsg1-1)
+(kicad_pcb (version 20171130) (host pcbnew 5.1.5-52549c5~84~ubuntu18.04.1)
   (general
     (thickness 1.6)
@@
   (page A4)
   (layers
-    (0 F.Cu signal)
-    (31 B.Cu signal)
+    (0 F.Cu signal hide)
+    (31 B.Cu signal hide)
     (32 B.Adhes user hide)
     (33 F.Adhes user hide)
@@
     (37 F.SilkS user hide)
     (38 B.Mask user hide)
-    (39 F.Mask user)
+    (39 F.Mask user hide)
     (40 Dwgs.User user hide)
     (41 Cmts.User user hide)
@@
       (net 7 /CATHODE))
   )
-  (gr_text "tom@tomk.in v1.0" (at 52.71 88.64 89) (layer B.SilkS)
+  (gr_text "tom@tomk.in v1.1" (at 52.71 88.64 89) (layer B.SilkS)
     (effects (font (size 1.8 1.8) (thickness 0.2)) (justify mirror))
   )
@@
       )
     )
+  )
+  (zone (net 0) (net_name "") (layer B.Mask) (hatch edge 0.508)
+    (connect_pads (clearance 0.508))
+    (min_thickness 0.254)
+    (fill yes (arc_segments 32) (thermal_gap 0.508) (thermal_bridge_width 0.508))
+    (polygon
+      (pts
+        (xy 71.5 117.75) (xy 19.75 118) (xy 20 24.75) (xy 71.75 24.25)
+      )
+    )
