File: 2021-xmas-tree/2021-xmas-tree.kicad_pcb (KiCad board)
At the start: 2 copper layers, 100 x 140.9 mm, 6 parts

Commit message: 2021-xmas-tree-2020Dec: reduced to 100mm size to save $$
Parts:
- moved G*** 177.5 mm to (100.0, 100.0) (x6)
Other:
- board size 100 x 140.9 mm -> 70.9 x 99.8 mm
- rule pad_to_mask_clearance: 0.05 -> 0
