File: syzygy-serdes-breakout/syzygy-serdes-breakout.sch (KiCad schematic (older format))
At the start: 18 parts, among them J1 QTH-020-01-X-D-DP-A, J2 USB3_A, J3 PMOD-2x6-FEMALE, J4 USB3_A_AS_PCIE, SW1 SW_DPDT_x2

Commit message: syzygy-serdes-breakout: fix missing ground pour on In1
Parts:
- added C6: 10uF/10V, tom-passives:C_0603_1608Metric, symbol tom-passives:C
- added C7: 0.1uF/10V, tom-passives:C_0603_1608Metric, symbol tom-passives:C
- added D2: LED, tom-opto:LED_0805_2012Metric, symbol tom-opto:LED
- added D3, D4: E6C1206RGBC3UDA, tom-opto:E6C1206RGBC3UDA, symbol tom-opto:E6C1206RGBC3UDA
- added J5: PMCU_SPI, tom-connectors:PinHeader_2x03_P2.54mm_Vertical, symbol tom-connectors:Conn_02x03_Odd_Even
- added R10: 1k, tom-passives:R_0603_1608Metric, symbol tom-passives:R
- added R11, R14: 1k2/5%, tom-passives:R_0603_1608Metric, symbol tom-passives:R
- added R12, R13, R15, R16: 300R/5%, tom-passives:R_0603_1608Metric, symbol tom-passives:R
- added R8: 10k/1%, tom-passives:C_0603_1608Metric, symbol tom-passives:R
- added R9: 10k/1%, tom-passives:R_0603_1608Metric, symbol tom-passives:R
- added U1: ATTINY44A-SSUR, tom-semiconductors:ATTINY44A-SSUR, symbol tom-semiconductors:ATTINY44A-SSUR
- R1, R5: value R -> 1M/5%
Connections:
- net +3V3: now also C7.1, D2.2 (A), J5.2 (Pin_2), R8.1, R9.1, U1.1 (VCC); no longer C2.1, J3.12 (VCC2), J3.6 (VCC1)
- net GND: now also C6.2, C7.2, J5.6 (Pin_6), U1.14 (GND)
- net R_GA: now also R9.2, U1.13 (PA0)
- net S10: now also R11.2
- net S11: now also R14.2
- net S12: now also R12.2
- net S13: now also R15.2
- net S14: now also R13.2
- net S15: now also R16.2
- net S2: now also J3.10 (D7); no longer J3.2 (D1)
- net S3: now also J3.9 (D6); no longer J3.1 (D0)
- net S8: now also J3.2 (D1); no longer J3.10 (D7)
- net S9: now also J3.1 (D0); no longer J3.9 (D6)
- net S0 renamed S0_N
- net S1 renamed S0_P
- net SCL renamed PMCU_SCK
- net PMCU_SCK: now also J5.3 (Pin_3), U1.9 (PA4)
- net SDA renamed PMCU_MOSI
- net PMCU_MOSI: now also J5.4 (Pin_4), U1.7 (PA6)
- net VIO1 renamed VCC
- net VCC: now also C2.1, J3.12 (VCC2), J3.6 (VCC1), C6.1, D3.2 (A), D4.2 (A)
- new net: D2.1 (K), R10.1
- new net: D3.1 (G), R13.1
- new net: D3.3 (R), R12.1
- new net: D3.4 (B), R11.1
- new net: D4.1 (G), R16.1
- new net: D4.3 (R), R15.1
- new net: D4.4 (B), R14.1
- new net PB2: R10.2, U1.5 (PB2)
- new net PMCU_MISO: J5.1 (Pin_1), U1.8 (PA5)
- new net PMCU_RESET: J5.5 (Pin_5), R8.2, U1.4 (PB3)
- no-connect marks 6 -> 18
Other:
- moved on the sheet: C3, C4
