File: peace-sign-sao/peace-sign.sch (KiCad schematic (older format))
At the start: 19 parts, among them X1 Badgelife_sao_connector_v169b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

Commit message: peace-sign-sao: change SAO connector back to 6 pin for stability
Parts:
- X1: footprint tom-connectors:Badgelife-SAOv169-SAO-2x3-SMD-NOCENTREPINS -> tom-connectors:Badgelife-SAOv169-SAO-2x3-SMD
Changed lines of the file:
@@
 F 0 "X1" H 3728 2696 50  0000 L CNN
 F 1 "Badgelife_sao_connector_v169bis" H 3728 2605 50  0000 L CNN
-F 2 "tom-connectors:Badgelife-SAOv169-SAO-2x3-SMD-NOCENTREPINS" H 3400 2850 50  0001 C CNN
+F 2 "tom-connectors:Badgelife-SAOv169-SAO-2x3-SMD" H 3400 2850 50  0001 C CNN
 F 3 "" H 3400 2850 50  0001 C CNN
 	1    3400 2650
