File: kindcalmsafe/kindcalmsafe.sch (KiCad schematic (older format))
At the start: 50 parts, among them X1 Badgelife_sao_connector_v169b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

Commit message: kindcalmsafe: commit unsaved schematic changes
Parts:
- gave numbers to parts that had none: 1
Changed lines of the file:
@@
 $EndComp
 $Comp
-L tom-mechanical:mech-only-no-pins H?
+L tom-mechanical:mech-only-no-pins H4
 U 1 1 600D7EA7
 P 9500 5900
-F 0 "H?" H 9525 5991 50  0000 L CNN
+F 0 "H4" H 9525 5991 50  0000 L CNN
 F 1 "kindcalmsafe-front-silk" H 9525 5900 50  0000 L CNN
 F 2 "kindcalmsafe:kindcalmsafe-silk-invert" H 9525 5809 50  0000 L CNN
