File: kindcalmsafe/kindcalmsafe.kicad_pcb (KiCad board)
At the start: 2 copper layers, 99.5 x 80.6 mm, 50 parts, among them X1 Badgelife_sao_connector_v169b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

Commit message: kindcalmsafe: fix 1204 led package
Parts:
- moved R4 3.49 mm to (142.6, 89.2), turned to 180 degrees
- moved R5 3.40 mm to (142.6, 86.9), turned to 180 degrees
- moved D26 1.00 mm to (85.0, 108.0)
Routing:
- net /BANK5: track 60.2 -> 94.9 mm
- net /BANK1: track 80.3 -> 71.4 mm
- net /BANK2: track 46.8 -> 55.2 mm
- net /BANK7: track 70.9 -> 65.4 mm
- net /BANK8: track 71.6 -> 76.8 mm
- net GND: track 519.9 -> 524.7 mm
- net /BANK9: track 47.0 -> 48.7 mm
- net /BANK6: track 59.7 -> 58.4 mm
- net /BANK4: track 49.7 -> 48.6 mm
- net /BANK3: track 74.9 -> 75.8 mm
