File: snoopy-sao/snoopy-sao/snoopy-sao.kicad_pcb (KiCad board)
At the start: 2 copper layers, 83.1 x 95.8 mm, 24 parts, among them X1 Badgelife_sao_connector_v169b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

Commit message: snoopy-sao: fix silk
Other:
- board text added: "JLCJLCJLCJLC"
- board text added: "Jan2021"
- board text added: "snoopy-sao @TomKeddie"
