File: blue-pill-bmp/hardware/blue-pill-bmp.sch (KiCad schematic (older format))
At the start: 36 parts, among them J2 USB_C_16PIN, J3 Conn_01x04, J4 Conn_02x05_SWD, SW1 SW_SPST, SW2 SW_DPDT_x2, U1 STM32F103C8T6, X1 8MHz, X2 32.768kHz

Commit message: blue-pill-bmp: add 2.54mm SWD connector
Parts:
- added J1: Conn_01x06, tom-connectors:PinHeader_1x06_P2.54mm_Vertical, symbol tom-connectors:Conn_01x06
Connections:
- net GND: now also J1.6 (Pin_6)
- net PA3: now also J1.1 (Pin_1)
- net PB4: now also J1.2 (Pin_2)
- net SWDCLK: now also J1.5 (Pin_5)
- net SWDIO: now also J1.4 (Pin_4)
- net VTARGET: now also J1.3 (Pin_3)
Other:
- moved on the sheet: C2, C3, J3
Changed lines of the file:
@@
 L power:GND #PWR0119
 U 1 1 5FDBC88D
-P 8500 3800
-F 0 "#PWR0119" H 8500 3550 50  0001 C CNN
-F 1 "GND" H 8505 3627 50  0000 C CNN
-F 2 "" H 8500 3800 50  0001 C CNN
-F 3 "" H 8500 3800 50  0001 C CNN
-	1    8500 3800
+P 8500 3350
+F 0 "#PWR0119" H 8500 3100 50  0001 C CNN
+F 1 "GND" H 8505 3177 50  0000 C CNN
+F 2 "" H 8500 3350 50  0001 C CNN
+F 3 "" H 8500 3350 50  0001 C CNN
+	1    8500 3350
 	1    0    0    -1
 $EndComp
@@
 L tom-connectors:Conn_01x04 J3
 U 1 1 5FE0F841
-P 8800 3500
-F 0 "J3" H 8880 3492 50  0000 L CNN
-F 1 "Conn_01x04" H 8880 3401 50  0000 L CNN
-F 2 "tom-connectors:PinHeader_1x04_P2.54mm_Vertical" H 8800 3500 50  0001 C CNN
-F 3 "~" H 8800 3500 50  0001 C CNN
-F 4 "DNP" H 8800 3500 50  0001 C CNN "LCSC"
-	1    8800 3500
+P 8800 3050
+F 0 "J3" H 8880 3042 50  0000 L CNN
+F 1 "Conn_01x04" H 8880 2951 50  0000 L CNN
+F 2 "tom-connectors:PinHeader_1x04_P2.54mm_Vertical" H 8800 3050 50  0001 C CNN
+F 3 "~" H 8800 3050 50  0001 C CNN
+F 4 "DNP" H 8800 3050 50  0001 C CNN "LCSC"
+	1    8800 3050
 	1    0    0    -1
 $EndComp
 Wire Wire Line
-	8600 3400 8500 3400
+	8600 2950 8500 2950
 Wire Wire Line
-	8500 3400 8500 3300
+	8500 2950 8500 2850
 Wire Wire Line
-	8600 3700 8500 3700
+	8600 3250 8500 3250
 Wire Wire Line
-	8500 3700 8500 3800
+	8500 3250 8500 3350
 Wire Wire Line
-	8600 3500 8450 3500
+	8600 3050 8450 3050
 Wire Wire Line
-	8600 3600 8450 3600
-Text Label 8450 3500 2    50   ~ 0
+	8600 3150 8450 3150
+Text Label 8450 3050 2    50   ~ 0
 PB6
-Text Label 8450 3600 2    50   ~ 0
+Text Label 8450 3150 2    50   ~ 0
 PB7
 Text Label 6400 3650 0    50   ~ 0
@@
 L tom-passives:C C2
 U 1 1 5FE89432
-P 7200 1750
-F 0 "C2" H 7315 1788 40  0000 L CNN
-F 1 "10uF/10V" H 7315 1712 40  0000 L CNN
-F 2 "tom-passives:C_0603_1608Metric" H 7315 1674 30  0001 L CNN
-F 3 "" H 7200 1750 60  0001 C CNN
-F 4 "C19702" V 7050 1750 40  0000 C CNN "LCSC"
-	1    7200 1750
+P 7400 1750
+F 0 "C2" H 7515 1788 40  0000 L CNN
+F 1 "10uF/10V" H 7515 1712 40  0000 L CNN
+F 2 "tom-passives:C_0603_1608Metric" H 7515 1674 30  0001 L CNN
+F 3 "" H 7400 1750 60  0001 C CNN
+F 4 "C19702" V 7250 1750 40  0000 C CNN "LCSC"
+	1    7400 1750
 	1    0    0    -1
 $EndComp
 Wire Wire Line
-	7200 1550 7200 1450
-Connection ~ 7200 1550
+	7400 1550 7400 1450
+Connection ~ 7400 1550
 Wire Wire Line
-	8800 1650 8800 1550
+	8600 1650 8600 1550
 $Comp
 L power:GND #PWR03
 U 1 1 5FE97E5D
-P 7200 1950
-F 0 "#PWR03" H 7200 1700 50  0001 C CNN
-F 1 "GND" H 7205 1777 50  0000 C CNN
-F 2 "" H 7200 1950 50  0001 C CNN
-F 3 "" H 7200 1950 50  0001 C CNN
-	1    7200 1950
+P 7400 1950
+F 0 "#PWR03" H 7400 1700 50  0001 C CNN
+F 1 "GND" H 7405 1777 50  0000 C CNN
+F 2 "" H 7400 1950 50  0001 C CNN
+F 3 "" H 7400 1950 50  0001 C CNN
+	1    7400 1950
 	1    0    0    -1
 $EndComp
 Wire Wire Line
-	8800 1550 9150 1550
+	8600 1550 8700 1550
 Wire Wire Line
-	9150 1550 9150 1450
+	8700 1550 8700 1450
 $Comp
 L power:+3.3V #PWR02
 U 1 1 5FE9B6AA
-P 9150 1450
-F 0 "#PWR02" H 9150 1300 50  0001 C CNN
-F 1 "+3.3V" H 9165 1623 50  0000 C CNN
-F 2 "" H 9150 1450 50  0001 C CNN
-F 3 "" H 9150 1450 50  0001 C CNN
-	1    9150 1450
+P 8700 1450
+F 0 "#PWR02" H 8700 1300 50  0001 C CNN
+F 1 "+3.3V" H 8715 1623 50  0000 C CNN
+F 2 "" H 8700 1450 50  0001 C CNN
+F 3 "" H 8700 1450 50  0001 C CNN
+	1    8700 1450
 	1    0    0    -1
 $EndComp
@@
 L power:GND #PWR04
 U 1 1 5FE9BE13
-P 9150 1950
-F 0 "#PWR04" H 9150 1700 50  0001 C CNN
-F 1 "GND" H 9155 1777 50  0000 C CNN
-F 2 "" H 9150 1950 50  0001 C CNN
-F 3 "" H 9150 1950 50  0001 C CNN
-	1    9150 1950
+P 8700 1950
+F 0 "#PWR04" H 8700 1700 50  0001 C CNN
+F 1 "GND" H 8705 1777 50  0000 C CNN
+F 2 "" H 8700 1950 50  0001 C CNN
+F 3 "" H 8700 1950 50  0001 C CNN
+	1    8700 1950
 	1    0    0    -1
 $EndComp
@@
 L tom-passives:CP_Small C3
 U 1 1 5FE9C6B8
-P 9150 1750
-F 0 "C3" H 9238 1834 50  0000 L CNN
-F 1 "100uF/6.3V" H 9238 1743 50  0000 L CNN
-F 2 "tom-passives:CP_EIA-3528-15_AVX-H" H 9150 1750 50  0001 C CNN
-F 3 "~" H 9150 1750 50  0001 C CNN
-F 4 "C16133" H 9238 1659 40  0000 L CNN "LCSC"
-	1    9150 1750
+P 8700 1750
+F 0 "C3" H 8788 1834 50  0000 L CNN
+F 1 "100uF/6.3V" H 8788 1743 50  0000 L CNN
+F 2 "tom-passives:CP_EIA-3528-15_AVX-H" H 8700 1750 50  0001 C CNN
+F 3 "~" H 8700 1750 50  0001 C CNN
+F 4 "C16133" H 8788 1659 40  0000 L CNN "LCSC"
+	1    8700 1750
 	1    0    0    -1
 $EndComp
 Wire Wire Line
-	9150 1550 9150 1650
-Connection ~ 9150 1550
+	8700 1550 8700 1650
+Connection ~ 8700 1550
 Wire Wire Line
-	9150 1850 9150 1950
+	8700 1850 8700 1950
 $Comp
 L power:+5V #PWR01
 U 1 1 5FEA6949
-P 7200 1450
-F 0 "#PWR01" H 7200 1300 50  0001 C CNN
-F 1 "+5V" H 7215 1623 50  0000 C CNN
-F 2 "" H 7200 1450 50  0001 C CNN
-F 3 "" H 7200 1450 50  0001 C CNN
-	1    7200 1450
+P 7400 1450
+F 0 "#PWR01" H 7400 1300 50  0001 C CNN
+F 1 "+5V" H 7415 1623 50  0000 C CNN
+F 2 "" H 7400 1450 50  0001 C CNN
+F 3 "" H 7400 1450 50  0001 C CNN
+	1    7400 1450
 	1    0    0    -1
 $EndComp
@@
 	0    1    1    0
 $EndComp
-Text Label 8500 3300 1    50   ~ 0
+Text Label 8500 2850 1    50   ~ 0
 VTARGET
 $Comp
-L power:GND #PWR?
+L power:GND #PWR05
 U 1 1 5FD9DEB6
-P 8100 2150
-F 0 "#PWR?" H 8100 1900 50  0001 C CNN
-F 1 "GND" H 8105 1977 50  0000 C CNN
-F 2 "" H 8100 2150 50  0001 C CNN
-F 3 "" H 8100 2150 50  0001 C CNN
-	1    8100 2150
+P 8100 1950
+F 0 "#PWR05" H 8100 1700 50  0001 C CNN
+F 1 "GND" H 8105 1777 50  0000 C CNN
+F 2 "" H 8100 1950 50  0001 C CNN
+F 3 "" H 8100 1950 50  0001 C CNN
+	1    8100 1950
 	1    0    0    -1
 $EndComp
-Connection ~ 8800 1550
+Connection ~ 8600 1550
 $Comp
 L tom-semiconductors:LM1117MPX-3.3 VR1
@@
 $EndComp
 Wire Wire Line
-	8800 1550 8600 1550
-Wire Wire Line
-	8800 1650 8600 1650
-Wire Wire Line
-	8100 1950 8100 2150
-Wire Wire Line
-	7200 1550 7600 1550
+	7400 1550 7600 1550
 $Bitmap
 Pos 9250 5350
@@
 EndData
 $EndBitmap
+$Comp
+L tom-connectors:Conn_01x06 J1
+U 1 1 5FDA305A
+P 8800 4300
+F 0 "J1" H 8880 4292 50  0000 L CNN
+F 1 "Conn_01x06" H 8880 4201 50  0000 L CNN
+F 2 "tom-connectors:PinHeader_1x06_P2.54mm_Vertical" H 8800 4300 50  0001 C CNN
+F 3 "~" H 8800 4300 50  0001 C CNN
+	1    8800 4300
+	1    0    0    -1
+$EndComp
+Wire Wire Line
+	8600 4100 8450 4100
+Text Label 8450 4100 2    50   ~ 0
+PA3
+Wire Wire Line
+	8600 4200 8450 4200
+Wire Wire Line
+	8600 4300 8150 4300
+Wire Wire Line
+	8150 4300 8150 4050
+Text Label 8150 4050 1    50   ~ 0
+VTARGET
+$Comp
+L power:GND #PWR08
+U 1 1 5FDB8ED5
+P 8450 4650
+F 0 "#PWR08" H 8450 4400 50  0001 C CNN
+F 1 "GND" H 8455 4477 50  0000 C CNN
+F 2 "" H 8450 4650 50  0001 C CNN
+F 3 "" H 8450 4650 50  0001 C CNN
+	1    8450 4650
+	1    0    0    -1
+$EndComp
+Wire Wire Line
+	8600 4600 8450 4600
+Wire Wire Line
+	8450 4600 8450 4650
+Wire Wire Line
+	8600 4500 8450 4500
+Wire Wire Line
+	8450 4400 8600 4400
+Text Label 8450 4400 2    50   ~ 0
+SWDIO
+Text Label 8450 4200 2    50   ~ 0
+PB4
+Text Label 8450 4500 2    50   ~ 0
+SWDCLK
 $EndSCHEMATC

Commit message: blue-pill-bmp: as submitted
Parts:
- VR1: footprint VREG_LM1117MPX-3.3 -> tom-semiconductors:VREG_LM1117MPX-3.3
Changed lines of the file:
@@
 F 0 "VR1" H 8100 2100 50  0000 C CNN
 F 1 "LM1117MPX-3.3" H 8100 2000 50  0000 C CNN
-F 2 "VREG_LM1117MPX-3.3" H 8100 1650 50  0001 L BNN
+F 2 "tom-semiconductors:VREG_LM1117MPX-3.3" H 8100 1650 50  0001 L BNN
 F 3 "" H 8100 1650 50  0001 L BNN
 F 4 "1.80 mm" H 8100 1650 50  0001 L BNN "MAXIMUM_PACKAGE_HEIGHT"
