File: ft4232h-breakout/ft4232h-breakout.kicad_pcb (KiCad board)
At the start: 2 copper layers, 64.1 x 47 mm, 18 parts, among them J1 Conn_01x03, J2 Conn_01x03, J3 Conn_01x03, J4 Conn_01x03, J5 Conn_02x05_SWD, J6 Conn_01x07, J7 Conn_01x07, J8 Conn_01x06, J9 Conn_01x02, X1 FT4232H-MODULE

Commit message: ft4232h-breakout: may release - change to SMTSO-M3 standoff
Parts:
- TP1: footprint tom-mechanical:STUD_SOLDER_M3 -> tom-mechanical:STUD_SOLDER_SMTSO_M3
Other:
- board text added: "@TomKeddie ft4232h-breakout May2021"
- board text removed: "@TomKeddie ft4232h-breakout Apr2021"
Changed lines of the file:
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@@
   (page A4)
   (title_block
-    (date 2021-04-18)
-    (rev Apr2021)
+    (date 2021-05-29)
+    (rev May2021)
   )
   (layers
@@
     (add_net "Net-(X1-Pad3-9)")
   )
-  (module tom-mechanical:STUD_SOLDER_M3 (layer B.Cu)
+  (module tom-mechanical:STUD_SOLDER_SMTSO_M3 (layer B.Cu)
     (at 99.06 87.63)
+    (descr "SMD Standoff Aliexpress")
+    (attr smd)
     (fp_text reference TP1 (at 0 -0.5) (layer B.SilkS) hide
       (effects (font (size 1 1) (thickness 0.15)) (justify mirror))
     )
-    (fp_text value TestPoint (at 0 0.5) (layer B.Fab) hide
+    (fp_text value TestPoint (at 0 0.5) (layer B.Fab)
       (effects (font (size 1 1) (thickness 0.15)) (justify mirror))
     )
-    (pad 1 thru_hole circle (at 0 0) (size 2 2) (drill 0.85) (layers *.Cu *.Mask)
-      (net 2 GND))
-    (pad 1 smd circle (at 0 0) (size 8 8) (layers B.Cu B.Paste B.Mask)
-      (net 2 GND))
+    (pad 1 thru_hole circle (at 0 0) (size 7 7) (drill 4.5) (layers *.Cu *.Mask)
+      (net 2 GND))
+    (model /home/tom/git/TomKeddie/prj-pcb-experiments/tom-kicad/footprints/3dmodels/SMTSO-M3-10ET-PennEngineering-3D-05-29-2021.stp
+      (offset (xyz 0 0 -1.6))
+      (scale (xyz 1 1 1))
+      (rotate (xyz 0 90 0))
+    )
   )
   (module tom-passives:R_0805_2012Metric (layer F.Cu)
@@
     (effects (font (size 1.9 1.9) (thickness 0.4)))
   )
-  (gr_text "@TomKeddie\nft4232h-breakout\nApr2021" (at 98.425 106.68 90) (layer B.SilkS)
+  (gr_text "@TomKeddie\nft4232h-breakout\nMay2021" (at 98.425 106.68 90) (layer B.SilkS)
     (effects (font (size 2 2) (thickness 0.4)) (justify mirror))
   )
