File: ch348_octo_serial/ch348_octo_serial.kicad_sch (KiCad schematic)
At the start: 49 parts, among them J1 USB_C_Receptacle_USB2.0, J2 Conn_01x01, J3 Conn_01x01, J4 Conn_01x01, J5 Conn_01x01, J6 VEXT, SW1 SW_DP4T, U1 CH348L, X1 8MHz

Commit message: ch348_octo_serial: fully routed, silk pending
Parts:
- R16: LCSC C17168 -> DNP
Connections:
- net TEST: now reaches R12.2, U1.94 (TEST)
- net XI: now reaches C8.1, U1.12 (XI), X1.1
- net XO: now reaches C9.1, U1.13 (XO), X1.2
- net RESET: now reaches C7.1, R10.2, U1.14 (RESET)
- net ACT: now reaches D2.1 (K), U1.29 (ACT)
- net CFG: now reaches R13.2, U1.7 (CFG)
- net TX_S: now reaches R15.1, U1.76 (TX_S)
- net RX_S: now reaches R14.1, U1.77 (RX_S)
Other:
- moved on the sheet: D2, R11, R12, R13

Commit message: ch348_octo_serial: Dec2022 as submitted
Parts:
- added H1: Front Octopus, ch348_octo_serial:octopus, symbol tom-mechanical:mech-only-no-pins
- added H2: Back Octopus, ch348_octo_serial:octopus_120, symbol tom-mechanical:mech-only-no-pins
Changed lines of the file:
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@@
     (pin "2")
+  )
+  (symbol (lib_id "tom-mechanical:mech-only-no-pins") (at 245.745 172.085 0) (unit 1)
+    (in_bom yes) (on_board yes) (fields_autoplaced)
+    (property "Reference" "H1" (id 0) (at 246.38 170.8149 0)
+      (effects (font (size 1.27 1.27)) (justify left))
+    )
+    (property "Value" "Front Octopus" (id 1) (at 246.38 173.3549 0)
+      (effects (font (size 1.27 1.27)) (justify left))
+    )
+    (property "Footprint" "ch348_octo_serial:octopus" (id 2) (at 245.745 172.085 0)
+      (effects (font (size 1.27 1.27)) hide)
+    )
+    (property "Datasheet" "" (id 3) (at 245.745 172.085 0)
+      (effects (font (size 1.27 1.27)) hide)
+    )
   )
   (symbol (lib_id "tom-connectors:Conn_01x01") (at 224.155 172.085 0) (unit 1)
@@
   (symbol (lib_id "power:GND") (at 180.975 48.26 90) (unit 1)
     (in_bom yes) (on_board yes)
-    (property "Reference" "#PWR032" (id 0) (at 187.325 48.26 0)
+    (property "Reference" "#PWR033" (id 0) (at 187.325 48.26 0)
       (effects (font (size 1.27 1.27)) hide)
     )
@@
     (pin "1")
     (pin "2")
+  )
+  (symbol (lib_id "tom-mechanical:mech-only-no-pins") (at 263.525 172.085 0) (unit 1)
+    (in_bom yes) (on_board yes) (fields_autoplaced)
+    (property "Reference" "H2" (id 0) (at 264.16 170.8149 0)
+      (effects (font (size 1.27 1.27)) (justify left))
+    )
+    (property "Value" "Back Octopus" (id 1) (at 264.16 173.3549 0)
+      (effects (font (size 1.27 1.27)) (justify left))
+    )
+    (property "Footprint" "ch348_octo_serial:octopus_120" (id 2) (at 263.525 172.085 0)
+      (effects (font (size 1.27 1.27)) hide)
+    )
+    (property "Datasheet" "" (id 3) (at 263.525 172.085 0)
+      (effects (font (size 1.27 1.27)) hide)
+    )
   )
   (symbol (lib_id "power:+2V5") (at 259.08 86.995 0) (unit 1)
@@
   (symbol (lib_id "power:GND") (at 189.865 27.94 0) (unit 1)
     (in_bom yes) (on_board yes)
-    (property "Reference" "#PWR035" (id 0) (at 189.865 34.29 0)
+    (property "Reference" "#PWR034" (id 0) (at 189.865 34.29 0)
       (effects (font (size 1.27 1.27)) hide)
     )
@@
   (symbol (lib_id "power:GND") (at 174.625 27.94 0) (unit 1)
     (in_bom yes) (on_board yes)
-    (property "Reference" "#PWR033" (id 0) (at 174.625 34.29 0)
+    (property "Reference" "#PWR032" (id 0) (at 174.625 34.29 0)
       (effects (font (size 1.27 1.27)) hide)
     )
@@
   (symbol (lib_id "power:GND") (at 192.405 45.72 90) (unit 1)
     (in_bom yes) (on_board yes)
-    (property "Reference" "#PWR034" (id 0) (at 198.755 45.72 0)
+    (property "Reference" "#PWR035" (id 0) (at 198.755 45.72 0)
       (effects (font (size 1.27 1.27)) hide)
     )
@@
       (reference "#PWR031") (unit 1) (value "+3.3V") (footprint "")
     )
+    (path "/a2226f90-feb8-47b5-8281-3a3c2cdf2fe5"
+      (reference "#PWR032") (unit 1) (value "GND") (footprint "")
+    )
     (path "/54566073-a62a-4a49-be08-980d88e1243c"
-      (reference "#PWR032") (unit 1) (value "GND") (footprint "")
-    )
-    (path "/a2226f90-feb8-47b5-8281-3a3c2cdf2fe5"
       (reference "#PWR033") (unit 1) (value "GND") (footprint "")
     )
+    (path "/909a2bc2-c3e5-422d-93af-c0a86268267b"
+      (reference "#PWR034") (unit 1) (value "GND") (footprint "")
+    )
     (path "/b510a78a-55bd-4d15-be8c-0aa2330031df"
-      (reference "#PWR034") (unit 1) (value "GND") (footprint "")
-    )
-    (path "/909a2bc2-c3e5-422d-93af-c0a86268267b"
       (reference "#PWR035") (unit 1) (value "GND") (footprint "")
     )
@@
       (reference "D4") (unit 1) (value "GREEN") (footprint "tom-opto:LED_0603_1608Metric")
     )
+    (path "/15bddf37-dc29-4d69-a259-f9180086fa04"
+      (reference "H1") (unit 1) (value "Front Octopus") (footprint "ch348_octo_serial:octopus")
+    )
+    (path "/69383d1a-b9b0-44c2-8864-b03863b50223"
+      (reference "H2") (unit 1) (value "Back Octopus") (footprint "ch348_octo_serial:octopus_120")
+    )
     (path "/8f01758d-3dc3-4cba-9a53-ecb070228d1c"
