File: ch348_octo_serial/serial-connectors.kicad_sch (KiCad schematic)
At the start: 3 parts, among them J15 JLCPCB_3.5MM_SOCKET_C18166, J16 Conn_01x07

Commit message: ch348_octo_serial: Dec2022 as submitted
Parts:
- J16: LCSC (none) -> C492415
Changed lines of the file:
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@@
+      (effects (font (size 1.27 1.27)) hide)
+    )
+    (property "LCSC" "C492415" (id 4) (at 95.885 74.295 0)
       (effects (font (size 1.27 1.27)) hide)
     )
