File: covid-dude/covid-dude.kicad_pcb (KiCad board)
At the start: 2 copper layers, 62.2 x 69.4 mm, 17 parts, among them X1 Badgelife_sao_connector_v169b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

Commit message: covid-dude: add JLCJLC text
Other:
- board text added: "covid-dude @TomKeddie Dec2022 JLCJLCJLCJLC"
- board text removed: "covid-dude @TomKeddie Dec2022"
Changed lines of the file:
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@@
   )
   (gr_line (start 98.7 92.4) (end 98.7 144) (layer "Dwgs.User") (width 0.15))
-  (gr_text "covid-dude\n@TomKeddie\nDec2022" (at 98.7 83.2) (layer "B.SilkS")
+  (gr_text "covid-dude\n@TomKeddie\nDec2022\nJLCJLCJLCJLC" (at 98.7 82.3) (layer "B.SilkS")
     (effects (font (size 3 3) (thickness 0.5)) (justify mirror))
   )
