File: esp8266-plugpack/esp8266-plugpack.kicad_pcb (KiCad board)
At the start: 2 copper layers, 44 x 71 mm, 45 parts, among them J1 Conn_01x04, J2 Conn_01x04, J3 Conn_01x02, U1 LTV-826S, U2 ESP-12, U3 AP2112K-3.3, U4 LTV-826S, U5 74LVC1G125, X1 HLK-PM01/03

Commit message: esp8266-plugpack: Apr2023 release
Other:
- board text added: "esp8266-plugpack @TomKeddie Apr2023"
