File: esp8266-plugpack/esp8266-plugpack.kicad_sch (KiCad schematic)
At the start: 37 parts, among them J1 Conn_01x04, J3 Conn_01x02, U1 LTV-826S, U2 ESP-12, U3 AP2112K-3.3, U4 LTV-826S, U5 74LVC1G125, X1 HLK-PM01/03

Commit message: esp8266-plugpack: placed and routed
Parts:
- removed C2: 100nF,16V,X7R, library:C_0402_1005Metric, symbol library:100nF,16V,X7R
- added C2: 100nF,50V,X7R, tom-passives:C_0603_1608Metric, symbol jlcpcb-basic-capacitor-0603:100nF,50V,X7R
- added C4: 10uF,10V,X5R, C_0603_1608Metric, symbol jlcpcb-basic-capacitor-0603:10uF,10V,X5R
- added H1: PCB OUTLINE, tom-mechanical:PCB_ALIEXPRESS_PLUGPACK_1, symbol tom-mechanical:mech-only-no-pins
- added J2: Conn_01x04, tom-connectors:JST_PH_B4B-PH-SM4-TB_1x04-1MP_P2.00mm_Vertical, symbol tom-connectors:Conn_01x04
- added R18, R19, R20, R21, R22: 0, tom-passives:R_0603_1608Metric, symbol jlcpcb-basic-resistor-0603:0
- C1, C3, C5: footprint C_0603_1608Metric -> tom-passives:C_0603_1608Metric
- D1: footprint (none) -> tom-semiconductors:Diode_Bridge_MBnnS; symbol tom-passives:BRIDGE -> tom-passives:BRIDGE_MBnnS
- D2: footprint (none) -> tom-opto:LED_0805_2012Metric
- D7: footprint (none) -> tom-opto:LED_D5.0mm-4_RGB
- F1: footprint (none) -> tom-passives:Fuse_2410
- F2: footprint (none) -> tom-passives:R_Axial_DIN0204_L3.6mm_D1.6mm_P7.62mm_Horizontal
- R1, R10, R11, R12, R13, R14, R15, R16, R17, R2, R3, R4, R5, R6, R7, R8, R9: footprint R_0603_1608Metric -> tom-passives:R_0603_1608Metric
- RV1: value Varistor -> MOV-10D561K; footprint (none) -> tom-passives:RV_Disc_D12mm_W3.9mm_P7.5mm
- TP1, TP2: footprint (none) -> tom-mechanical:TestPoint_Pad_D3.0mm
- U2: footprint ESP8266:ESP-12E_SMD -> tom-modules:ESP-12E_SMD
- U5: footprint library:SOT-23-5 -> tom-semiconductors:SOT-23-5
- X1: footprint (none) -> tom-modules:HLK-PMxx
Connections:
- net +3.3V: now also D7.2 (A), C4.1; no longer D7.4 (A)
- net +5V: now also C2.1
- net AC16A: now also R18.1
- net AC16B: now also D1.3, R21.1; no longer D1.2
- net DC12OUT: now also R20.1
- net DC12OUT_5V: now also R22.1
- net DC14IN: now also R19.1
- net GND: now also C2.2, C4.2, J2.4 (Pin_4)
- net VCC: now reaches R16.1, R17.1, X1.4 (DCOUT)
- net VCC: now also J2.1 (Pin_1)
- net at R8.2: now also D1.2 (-); no longer D1.1 (-)
- net at R2.1: now also D7.4 (BK); no longer D7.3 (BK)
- net at R5.1: now also D1.1 (+); no longer D1.3 (+)
- net at R7.1: now also D7.3 (GK); no longer D7.2 (GK)
- new net: J2.2 (Pin_2), R18.2, R19.2
- new net: J2.3 (Pin_3), R20.2, R21.2, R22.2

Commit message: esp8266-plugpack: Apr2023 release
Parts:
- U2: LCSC (none) -> C82891
Changed lines of the file:
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@@
+      (effects (font (size 1.27 1.27)) hide)
+    )
+    (property "LCSC" "C82891" (at 180.34 96.52 0)
       (effects (font (size 1.27 1.27)) hide)
     )
