File: mikrobus-pmod-adapt/mikrobus-pmod-adapt.kicad_pcb (KiCad board)
At the start: 2 copper layers, 25.4 x 28.6 mm, 17 parts, among them J1 PMOD-2x6-FEMALE

Commit message: mikrobus-pmod: change to 16 poin connector
Parts:
- removed ALTD0, ALTD1, ALTD2, ALTD3: SolderJumper_2_Open, tom-mechanical:SolderJumper-2_P1.3mm_Open_Pad1.0x1.5mm
- removed D0, D1, D2, D3, D4, D5, D6, D7: BRIDGED, tom-mechanical:SolderJumper-2_P1.3mm_Bridged_Pad1.0x1.5mm
- removed J1: PMOD-2x6-FEMALE, tom-connectors:PMOD_2X6_PTH_RA_SOCKET
- added J2: PMOD++, tom-connectors:PMOD_2x8_PTH_RA_SOCKET, F.Cu at (108.9, 84.0)
- U1: footprint tom-modules:MIKROBUS_ADD_ON_SMALL -> tom-modules:MIKROBUS_ADD_ON_MEDIUM
- moved LED1 25.4 mm to (100.0, 111.8), turned to 0 degrees
- moved R1 25.4 mm to (100.0, 111.8), turned to 0 degrees
- moved C1 21.0 mm to (90.2, 90.8), turned to 180 degrees
Connections:
- U1 pad A1: /MD8 -> /A1
- U1 pad A2: /MD9 -> /A2
- U1 pad A3: /MD0 -> /A3
- U1 pad A4: /MD3 -> /A4
- U1 pad A5: /MD2 -> /A5
- U1 pad A6: /MD1 -> /A6
- U1 pad B1: /MD10 -> /B1
- U1 pad B2: /MD11 -> /B2
- U1 pad B3: /MD4 -> /B3
- U1 pad B4: /MD5 -> /B4
- U1 pad B5: /MD6 -> /B5
- U1 pad B6: /MD7 -> /B6
Routing:
- net /B6: track 0.00 -> 38.6 mm, vias 0 -> 1
- net /B5: track 0.00 -> 33.6 mm, vias 0 -> 1
- net /B4: track 0.00 -> 28.1 mm, vias 0 -> 1
- net /A3: track 0.00 -> 27.1 mm, vias 0 -> 1
- net /A5: track 0.00 -> 27.1 mm, vias 0 -> 1
- net /A4: track 0.00 -> 27.1 mm, vias 0 -> 1
- net /A2: track 0.00 -> 27.1 mm, vias 0 -> 1
- net /A6: track 0.00 -> 26.7 mm, vias 0 -> 1
- net /MD10: track 26.5 -> 0.00 mm, vias 1 -> 0
- net /A1: track 0.00 -> 25.6 mm
- net /MD9: track 24.8 -> 0.00 mm, vias 2 -> 0
- net /B3: track 0.00 -> 23.0 mm, vias 0 -> 1
- net /MD4: track 22.8 -> 0.00 mm, vias 1 -> 0
- net /MD8: track 22.3 -> 0.00 mm, vias 1 -> 0
- net /MD11: track 22.2 -> 0.00 mm, vias 2 -> 0
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- added copper zone on F.Cu, net GND
Other:
- board size 25.4 x 28.6 mm -> 25.4 x 42.9 mm
- board text added: "@TomKeddie Mar2024 mikrobus pmod adapt"
- board text removed: "@TomKeddie Jan2024 mikrobus pmod adapt"
