File: mikrobus-pmod-adapt/mikrobus-pmod-adapt.kicad_sch (KiCad schematic)
At the start: 17 parts, among them J1 PMOD-2x6-FEMALE

Commit message: mikrobus-pmod: change to 16 poin connector
Parts:
- removed ALTD0, ALTD1, ALTD2, ALTD3: SolderJumper_2_Open, tom-mechanical:SolderJumper-2_P1.3mm_Open_Pad1.0x1.5mm, symbol tom-mechanical:SolderJumper_2_Open
- removed D0, D1, D2, D3, D4, D5, D6, D7: BRIDGED, tom-mechanical:SolderJumper-2_P1.3mm_Bridged_Pad1.0x1.5mm, symbol tom-mechanical:SolderJumper_2_Bridged
- removed J1: PMOD-2x6-FEMALE, tom-connectors:PMOD_2X6_PTH_RA_SOCKET, symbol tom-connectors:PMOD-2x6-FEMALE
- added J2: PMOD++, tom-connectors:PMOD_2x8_PTH_RA_SOCKET, symbol Connector_Generic:Conn_02x08_Top_Bottom
Connections:
- net +3.3V: now also J2.16 (Pin_16), J2.8 (Pin_8)
- net GND: now also J2.15 (Pin_15), J2.7 (Pin_7)
- net MD0 renamed A3
- net A3: now also J2.3 (Pin_3)
- net MD1 renamed A6
- net A6: now also J2.6 (Pin_6)
- net MD10 renamed B1
- net B1: now also J2.9 (Pin_9)
- net MD11 renamed B2
- net B2: now also J2.10 (Pin_10)
- net MD2 renamed A5
- net A5: now also J2.5 (Pin_5)
- net MD3 renamed A4
- net A4: now also J2.4 (Pin_4)
- net MD4 renamed B3
- net B3: now also J2.11 (Pin_11)
- net MD5 renamed B4
- net B4: now also J2.12 (Pin_12)
- net MD6 renamed B5
- net B5: now also J2.13 (Pin_13)
- net MD7 renamed B6
- net B6: now also J2.14 (Pin_14)
- net MD8 renamed A1
- net A1: now also J2.1 (Pin_1)
- net MD9 renamed A2
- net A2: now also J2.2 (Pin_2)
