File: 2024-supercon-sign-sao/2024-supercon-sign-sao.kicad_pcb (KiCad board)
At the start: 2 copper layers, 66 x 75 mm, 137 parts, among them J1 Conn_01x06, Q1 AO3400A, Q2 AO3400A, Q3 AO3400A, U1 CH32V003F4P6

Commit message: 2024-supercon-sign-sao: add bottom silk
Other:
- board text added: "@TomKeddie Nov2024 2024-supercon-sign-sao https://github.com/TomKeddie/prj-pcb-experiments"
Changed lines of the file:
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@@
 		(tags "resistor")
 		(property "Reference" "R63"
-			(at 0 0 0)
+			(at 0 0.25 0)
 			(layer "B.SilkS")
 			(effects
@@
 		(tags "resistor")
 		(property "Reference" "R62"
-			(at 0 0 0)
+			(at 0 0.25 0)
 			(layer "B.SilkS")
 			(effects
@@
 		)
 	)
+	(gr_text "@TomKeddie\nNov2024\n2024-supercon-sign-sao\nhttps://github.com/TomKeddie/prj-pcb-experiments"
+		(at 122 96 45)
+		(layer "B.SilkS")
+		(effects
+			(font
+				(size 2 2)
+				(thickness 0.25)
+			)
+			(justify mirror)
+		)
+	)
