File: 2024-rfid-sao/2024-rfid-sao.kicad_sch (KiCad schematic)
At the start: 9 parts, among them U1 M24LR64E, X1 Badgelife_sao_connector_v169b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

Commit message: 2024-rfid-sao: updates for jlcpcb
Parts:
- C2: LCSC C344190 -> C1525
Changed lines of the file:
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@@
+			)
+		)
+		(property "Field6" ""
+			(at 118.11 96.52 0)
+			(effects
+				(font
+					(size 1.27 1.27)
+				)
+				(hide yes)
 			)
 		)
@@
 			)
 		)
-		(property "LCSC" "C344190"
-			(at 58.42 95.25 0)
-			(effects
+		(property "LCSC" "C1525"
+			(at 58.42 95.25 0)
+			(effects

Commit message: 2024-rfid-sao: change RFID chip to 4k version
Parts:
- U1: LCSC C2649483 -> C157372
Changed lines of the file:
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@@
 			)
 		)
-		(property "LCSC" "C2649483"
+		(property "LCSC" "C157372"
 			(at 118.11 96.52 0)
 			(effects
