File: 2025-usb-pd-plank/kicad/usb-pd-plank.kicad_sch (KiCad schematic)
At the start: 37 parts, among them J1 USB_C_Receptacle_USB2.0_16P, J2 USB_C_Receptacle_USB2.0_16P, J3 Bus Pirate, J4 Bus Pirate, J5 LINK, Q1 AO3400A, Q2 AO3400A, Q3 AO3400A, Q4 AO3400A, U1 PTN5110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

Commit message: 2025-usb-pd-plank: placed and routed
Parts:
- removed U2, U3: NX20P5090, lib:WLCSP-15_3x5_B1.54_2.56mm_P0.5mm, symbol lib:NX20P5090
- added Q5, Q6, Q7, Q8: AO4407A, lib:SO-8_3.9x4.9mm_P1.27mm, symbol lib:AO4407A
- added R12, R15: 100k, lib:R_0402_1005Metric, symbol library:100k
- added R13, R14: 10k, lib:R_0402_1005Metric, symbol lib:R_Small
- U1: now fitted; now in the parts list
Connections:
- net +5V: now also Q7.5 (D), Q7.6 (D), Q7.7 (D), Q7.8 (D)
- net EN_SRC: now also J3.4 (Pin_4), J4.4 (Pin_4); no longer J3.6 (Pin_6), J4.6 (Pin_6)
- net USBIN_CC1: no longer D2.5 (A)
- net USBIN_CC2: no longer D1.5 (A)
- net USBIN_VBUS: now also Q5.5 (D), Q5.6 (D), Q5.7 (D), Q5.8 (D)
- net USBOUT_VBUS: now also Q6.5 (D), Q6.6 (D), Q6.7 (D), Q6.8 (D), Q8.5 (D), Q8.6 (D), Q8.7 (D), Q8.8 (D)
- net ~{ALERT}: now also J3.6 (Pin_6), J4.6 (Pin_6); no longer J3.4 (Pin_4), J4.4 (Pin_4)
- net ~{EN_SNK}: now also R14.2
- net ~{EN_SRC}: now also R13.2
- new net: Q7.1 (S), Q7.2 (S), Q7.3 (S), Q8.1 (S), Q8.2 (S), Q8.3 (S), R15.1
- new net: Q7.4 (G), Q8.4 (G), R14.1, R15.2
- new net: Q5.1 (S), Q5.2 (S), Q5.3 (S), Q6.1 (S), Q6.2 (S), Q6.3 (S), R12.1
- new net: Q5.4 (G), Q6.4 (G), R12.2, R13.1
Other:
- moved on the sheet: R5, R7

Commit message: 2025-usb-pd-plank: read for mfg
Changed i2c resistors to 10k
Changed all LEDs to green
Changed all power caps to 4.7uF/50V
(cost reduction by $us10)
Parts:
- C1, C2, C3: value 2.2uF/16V -> 4.7uF/50V; footprint lib:C_0603_1608Metric -> lib:C_1206_3216Metric; LCSC C23630 -> C29823
- C5: value 1uF/50V -> 4.7uF/50V; LCSC C1848 -> C29823
- D3: value RED -> GREEN; LCSC C84256 -> C2297
- D5: value YELLOW -> GREEN; LCSC C2296 -> C2297
- J3, J5: now left out of the parts list
- R1, R2: value 4.7k -> 10k; LCSC C23162 -> C25744
Other:
- note added: "Note that caps on PD IC are out of spec to reduce part count."
Changed lines of the file:
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@@
 	(generator_version "9.0")
 	(paper "A4")
+	(text "Note that caps on PD IC are out of spec to reduce part count."
+		(exclude_from_sim no)
+		(at 137.16 59.69 0)
+		(effects
+			(font
+				(size 1.27 1.27)
+			)
+		)
+	)
 	(text "- Source and Sink connectors\n- Function as PD sink with VBUS on terminal\n- Function as Source for PD query only (5v)\n- Function as tap for PD exchange"
 		(exclude_from_sim no)
@@
 			)
 		)
-		(property "Value" "2.2uF/16V"
+		(property "Value" "4.7uF/50V"
 			(at 149.86 77.4762 0)
 			(effects
@@
 			)
 		)
-		(property "Footprint" "lib:C_0603_1608Metric"
+		(property "Footprint" "lib:C_1206_3216Metric"
 			(at 147.32 76.2 0)
 			(effects
@@
 			)
 		)
-		(property "LCSC" "C23630"
+		(property "LCSC" "C29823"
 			(at 147.32 76.2 0)
 			(effects
@@
 			)
 		)
-		(property "Value" "2.2uF/16V"
+		(property "Value" "4.7uF/50V"
 			(at 161.2963 82.55 90)
 			(effects
@@
 			)
 		)
-		(property "Footprint" "lib:C_0603_1608Metric"
+		(property "Footprint" "lib:C_1206_3216Metric"
 			(at 161.29 86.36 0)
 			(effects
@@
 			)
 		)
-		(property "LCSC" "C23630"
+		(property "LCSC" "C29823"
 			(at 161.29 86.36 0)
 			(effects
@@
 			)
 		)
-		(property "Value" "1uF/50V"
+		(property "Value" "4.7uF/50V"
 			(at 69.85 85.0962 0)
 			(effects
@@
 			)
 		)
-		(property "LCSC" "C1848"
+		(property "LCSC" "C29823"
 			(at 67.31 83.82 0)
 			(effects
@@
 		(unit 1)
 		(exclude_from_sim no)
-		(in_bom yes)
+		(in_bom no)
 		(on_board yes)
 		(dnp no)
@@
 			)
 		)
-		(property "Value" "RED"
+		(property "Value" "GREEN"
 			(at 27.94 25.4 0)
 			(effects
@@
 			)
 		)
-		(property "LCSC" "C84256"
+		(property "LCSC" "C2297"
 			(at 30.48 25.4 0)
 			(effects
@@
 			)
 		)
-		(property "Value" "YELLOW"
+		(property "Value" "GREEN"
 			(at 66.04 170.18 0)
 			(effects
@@
 			)
 		)
-		(property "LCSC" "C2296"
+		(property "LCSC" "C2297"
 			(at 68.58 170.18 0)
 			(effects
@@
 			)
 		)
-		(property "Value" "2.2uF/16V"
+		(property "Value" "4.7uF/50V"
 			(at 127 77.4762 0)
 			(effects
@@
 			)
 		)
-		(property "Footprint" "lib:C_0603_1608Metric"
+		(property "Footprint" "lib:C_1206_3216Metric"
 			(at 129.54 76.2 0)
 			(effects
@@
 			)
 		)
-		(property "LCSC" "C23630"
+		(property "LCSC" "C29823"
 			(at 129.54 76.2 0)
 			(effects
@@
 			)
 		)
-		(property "Value" "4.7k"
+		(property "Value" "10k"
 			(at 76.2 26.67 0)
 			(effects
@@
 			)
 		)
-		(property "LCSC" "C23162"
+		(property "LCSC" "C25744"
 			(at 74.93 25.4 0)
 			(effects
@@
 			)
 		)
-		(property "Value" "4.7k"
+		(property "Value" "10k"
 			(at 68.58 26.67 0)
 			(effects
@@
 			)
 		)
-		(property "LCSC" "C23162"
+		(property "LCSC" "C25744"
 			(at 67.31 25.4 0)
 			(effects
@@
 		(unit 1)
 		(exclude_from_sim no)
-		(in_bom yes)
+		(in_bom no)
 		(on_board yes)
 		(dnp no)

Commit message: 2025-usb-pd-plank: add VBUS connector, silk fixes.  As submitted.
Parts:
- added J6: Conn_01x02, lib:JST_PH_S2B-PH-SM4-TB_1x02-1MP_P2.00mm_Horizontal, symbol lib:Conn_01x02
Connections:
- net GND: now also J6.2 (Pin_2)
- net USBOUT_VBUS: now also J6.1 (Pin_1)
Changed lines of the file:
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@@
+		)
+	)
+	(label "USBOUT_VBUS"
+		(at 203.2 135.89 180)
+		(effects
+			(font
+				(size 1.27 1.27)
+			)
+			(justify right bottom)
 		)
 	)
@@
 	)
 	(symbol
+		(lib_id "lib:Conn_01x02")
+		(at 208.28 135.89 0)
+		(unit 1)
+		(exclude_from_sim no)
+		(in_bom no)
+		(on_board yes)
+		(dnp yes)
+		(fields_autoplaced yes)
+		(property "Reference" "J6"
+			(at 210.82 135.8899 0)
+			(effects
+				(font
+					(size 1.27 1.27)
+				)
+				(justify left)
+			)
+		)
+		(property "Value" "Conn_01x02"
+			(at 210.82 138.4299 0)
+			(effects
+				(font
+					(size 1.27 1.27)
+				)
+				(justify left)
+			)
+		)
+		(property "Footprint" "lib:JST_PH_S2B-PH-SM4-TB_1x02-1MP_P2.00mm_Horizontal"
+			(at 208.28 135.89 0)
+			(effects
+				(font
+					(size 1.27 1.27)
+				)
+				(hide yes)
+			)
+		)
+		(property "Datasheet" "~"
+			(at 208.28 135.89 0)
+			(effects
+				(font
+					(size 1.27 1.27)
+				)
+				(hide yes)
+			)
+		)
+		(property "Description" "Generic connector, single row, 01x02, script generated (kicad-library-utils/schlib/autogen/connector/)"
+			(at 208.28 135.89 0)
+			(effects
+				(font
+					(size 1.27 1.27)
+				)
+				(hide yes)
+			)
+		)
+		(pin "2"
+		)
+		(pin "1"
+		)
+		(instances
+			(project ""
+				(path "/6a1536ac-06de-4a63-8df8-45f19360eb67"
+					(reference "J6")
+					(unit 1)
+				)
+			)
+		)
+	)
+	(symbol
 		(lib_id "library:100k")
 		(at 26.67 189.23 0)
@@
 					(unit 1)
 				)
+			)
+		)
+	)
+	(symbol
+		(lib_id "power:GND")
+		(at 203.2 138.43 0)
+		(unit 1)
+		(exclude_from_sim no)
+		(in_bom yes)
+		(on_board yes)
+		(dnp no)
+		(property "Reference" "#PWR031"
+			(at 203.2 144.78 0)
+			(effects
+				(font
+					(size 1.27 1.27)
+				)
+				(hide yes)
+			)
+		)
+		(property "Value" "GND"
+			(at 203.2 142.24 0)
+			(effects
+				(font
+					(size 1.27 1.27)
+				)
+			)
+		)
+		(property "Footprint" ""
+			(at 203.2 138.43 0)
+			(effects
+				(font
+					(size 1.27 1.27)
+				)
+				(hide yes)
+			)
+		)
+		(property "Datasheet" ""
+			(at 203.2 138.43 0)
+			(effects
+				(font
+					(size 1.27 1.27)
+				)
+				(hide yes)
+			)
+		)
+		(property "Description" "Power symbol creates a global label with name \"GND\" , ground"
+			(at 203.2 138.43 0)
+			(effects
+				(font
+					(size 1.27 1.27)
+				)
+				(hide yes)
+			)
+		)
+		(pin "1"
+		)
+		(instances
+			(project "usb-pd-plank"
+				(path "/6a1536ac-06de-4a63-8df8-45f19360eb67"
+					(reference "#PWR031")
+					(unit 1)
+				)
