File: 2024-led-ctrl-24v/kicad/led-ctrl-24v.kicad_sch (KiCad schematic)
At the start: 24 parts, among them J1 Conn_01x04, J2 Conn_01x02, J3 Conn_01x05, Q1 AO3400A, SW1 SW_Push_Dual, SW2 SW_Push_Dual, SW3 SW_Push_Dual, SW4 SW_Push_Dual, SW5 SW_Push_Dual, U2 ESP-12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

Commit message: led-ctrl-24v: progress checkin
Parts:
- removed C1: 10uF/10V/X5R, library:C_0603_1608Metric, symbol library:10uF,10V,X5R
- added C3: 10nF/50V/X7R, library:C_0402_1005Metric, symbol library:10nF/50V/X7R
- added C4: 10uF/50V/X5R, library:C_1206_3216Metric, symbol library:22uF/25V/X5R
- added C5: 220uF/6.3V/TANT, library:CP_EIA-3528-12_Kemet-T, symbol library:220uF/6.3V/TANT
- added C6, C7: 10uF/10V/X5R, library:C_0603_1608Metric, symbol library:10uF,10V,X5R
- added D1: B340, library:D_SMA, symbol library:B340
- added L1: 33uH/1A, library:CYA630, symbol library:L_CYA0630
- added R10: 0, library:R_0603_1608Metric, symbol library:0
- added R11, R15: 10k, library:R_0402_1005Metric, symbol library:10k
- added R13: 4.7k, library:R_0402_1005Metric, symbol library:10k
- added U1: TPS5430DDA, library:TI_SO-PowerPAD-8_ThermalVias, symbol library:TPS5430DDA
- added U3: XC6206P332MR-G, library:SOT-23, symbol library:XC6206P332MR-G
Connections:
- net +24V: now also C4.1, U1.7 (VIN)
- net +3.3V: now also C6.1, U3.2 (VO)
- net +5V: now also C7.1, R10.2, U3.3 (VI)
- net BTN0: no longer SW1.4
- net BTN1: no longer SW2.4
- net BTN2: no longer SW3.4
- net BTN3: no longer SW4.4
- net BTN4: no longer SW5.4
- net GND: now also C4.2, C5.2, C6.2, C7.2, D1.2 (A), R11.2, R13.2, U1.6 (GND), U1.9 (GNDPAD), U3.1 (GND); no longer SW1.3, SW2.3, SW3.3, SW4.3, SW5.3
- new net: C3.1, U1.1 (BOOT)
- new net PH: C3.2, D1.1 (K), L1.1, U1.8 (PH)
- new net VOUT: C5.1, L1.2, R10.1, R15.1
- new net VSENSE: R11.1, R13.1, R15.2, U1.4 (VSENSE)
- no-connect marks 2 -> 3
Other:
- moved on the sheet: C2, J1, J2, J3, Q1, R1, R12, R14, R2, R3, R4, R5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

Commit message: 2024-led-ctrl-24v: abandoned - too expensive
Parts:
- J2, J3, SW1, SW2, SW3, SW4, SW5: now not fitted; now left out of the parts list
Changed lines of the file:
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@@
 		(unit 1)
 		(exclude_from_sim no)
-		(in_bom yes)
+		(in_bom no)
 		(on_board yes)
-		(dnp no)
+		(dnp yes)
 		(property "Reference" "SW1"
 			(at 31.75 24.765 0)
@@
 		(unit 1)
 		(exclude_from_sim no)
-		(in_bom yes)
+		(in_bom no)
 		(on_board yes)
-		(dnp no)
+		(dnp yes)
 		(property "Reference" "SW3"
 			(at 31.75 50.165 0)
@@
 		(unit 1)
 		(exclude_from_sim no)
-		(in_bom yes)
+		(in_bom no)
 		(on_board yes)
-		(dnp no)
+		(dnp yes)
 		(property "Reference" "SW2"
 			(at 31.75 37.465 0)
@@
 		(unit 1)
 		(exclude_from_sim no)
-		(in_bom yes)
+		(in_bom no)
 		(on_board yes)
-		(dnp no)
+		(dnp yes)
 		(property "Reference" "SW5"
 			(at 31.75 75.565 0)
@@
 		(unit 1)
 		(exclude_from_sim no)
-		(in_bom yes)
+		(in_bom no)
 		(on_board yes)
-		(dnp no)
+		(dnp yes)
 		(fields_autoplaced yes)
 		(property "Reference" "J3"
@@
 		(unit 1)
 		(exclude_from_sim no)
-		(in_bom yes)
+		(in_bom no)
 		(on_board yes)
-		(dnp no)
+		(dnp yes)
 		(property "Reference" "SW4"
 			(at 31.75 62.865 0)
@@
 		(unit 1)
 		(exclude_from_sim no)
-		(in_bom yes)
+		(in_bom no)
 		(on_board yes)
-		(dnp no)
+		(dnp yes)
 		(property "Reference" "J2"
 			(at 22.86 97.79 0)
