File: 2024-clock-retrofit/kicad/2024-clock-retrofit.kicad_sch (KiCad schematic)
At the start: 40 parts, among them SW1 SW_Push, U1 TLC59025, U2 ESP32-WROOM-32, U3 TLC59025, U4 AZ1117-3.3

Commit message: Add misc files from x570
Changed lines of the file:
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@@
+		)
+	)
+	(polyline
+		(pts
+			(xy 175.26 33.02) (xy 185.42 33.02)
+		)
+		(stroke
+			(width 0)
+			(type dot)
 		)
 	)
@@
 		)
 	)
+	(polyline
+		(pts
+			(xy 175.26 43.18) (xy 185.42 43.18)
+		)
+		(stroke
+			(width 0)
+			(type dot)
+		)
+	)
 	(wire
 		(pts
@@
 		)
 	)
+	(polyline
+		(pts
+			(xy 185.42 22.86) (xy 185.42 58.42)
+		)
+		(stroke
+			(width 0)
+			(type dot)
+		)
+	)
 	(wire
 		(pts
@@
 		)
 	)
+	(polyline
+		(pts
+			(xy 175.26 22.86) (xy 185.42 22.86)
+		)
+		(stroke
+			(width 0)
+			(type dot)
+		)
+	)
 	(wire
 		(pts
@@
 		)
 	)
+	(polyline
+		(pts
+			(xy 175.26 53.34) (xy 185.42 53.34)
+		)
+		(stroke
+			(width 0)
+			(type dot)
+		)
+	)
