File: ft4232h-breakout/v3.x/ft4232h-breakout.kicad_pcb (KiCad board)
At the start: 2 copper layers, 83.2 x 57.8 mm, 73 parts, among them J1 Conn_01x03, J10 USB_C_Receptacle_USB2.0, J2 Conn_01x03, J3 Conn_01x03, J4 Conn_01x03, J5 JLCPCB_3.5MM_SOCKET_C18166, J6 JLCPCB_3.5MM_SOCKET_C18166, J7 JLCPCB_3.5MM_SOCKET_C18166, J8 JLCPCB_3.5MM_SOCKET_C18166, J9 USB_B_Micro, U1 74HC595, U2 FT4232H, U3 AT93C46DN-SH-T, X1 12MHz

Commit message: Add misc files from x570
Routing:
- net (no net): vias 0 -> 4
Other:
- board text added: "Quad USB Serial Jun2022 v3.1 @TomKeddie"
- board text removed: "Quad USB Serial V3.1 @TomKeddie"
Changed lines of the file:
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@@
     (property "Sheetname" "")
     (attr smd)
-    (fp_text reference "C21" (at -0.635 2.54 90) (layer "F.SilkS")
+    (fp_text reference "C21" (at -1.778 2.54 90) (layer "F.SilkS")
       (effects (font (size 1.5 1.5) (thickness 0.25)))
     )
@@
     (property "Sheetname" "")
     (attr smd)
-    (fp_text reference "R11" (at 3.14309 -1.347038 135) (layer "F.SilkS")
+    (fp_text reference "R11" (at 3.771708 -1.257236 135) (layer "F.SilkS")
       (effects (font (size 1.5 1.5) (thickness 0.25)))
     )
@@
     (property "Sheetname" "")
     (attr smd)
-    (fp_text reference "C6" (at -3.66 -1.905 90) (layer "F.SilkS")
+    (fp_text reference "C6" (at -0.231 -1.524 90) (layer "F.SilkS")
       (effects (font (size 1.5 1.5) (thickness 0.25)))
     )
@@
   (gr_line (start 141.58125 71.11875) (end 58.41875 71.11875) (layer "Edge.Cuts") (width 0.1))
   (gr_circle (center 138.1 74.6) (end 140.6 74.6) (layer "F.CrtYd") (width 0.1) (fill none))
-  (gr_circle (center 61.9 74.6) (end 65.9 74.6) (layer "F.CrtYd") (width 0.1) (fill none))
+  (gr_circle (center 61.9 74.6) (end 64.4 74.6) (layer "F.CrtYd") (width 0.1) (fill none))
   (gr_circle (center 61.9 125.4) (end 64.4 125.4) (layer "F.CrtYd") (width 0.1) (fill none))
   (gr_circle (center 138.1 125.4) (end 140.6 125.4) (layer "F.CrtYd") (width 0.1) (fill none))
@@
     (effects (font (size 4 4) (thickness 0.5)) (justify mirror))
   )
-  (gr_text "Quad USB Serial\nV3.1\n@TomKeddie" (at 73.152 88.646) (layer "F.SilkS")
+  (gr_text "Quad USB Serial\nJun2022\nv3.1\n@TomKeddie" (at 71.628 85.344) (layer "F.SilkS")
     (effects (font (size 2 2) (thickness 0.3)))
   )
@@
     (style (thickness 0.1) (arrow_length 1.27) (text_position_mode 0) (extension_height 0.58642) (extension_offset 0.5) keep_text_aligned)
   )
+  (via (at 138.1 74.6) (size 4) (drill 2.6) (layers "F.Cu" "B.Cu") (free) (net 0))
+  (via (at 61.9 125.4) (size 4) (drill 2.6) (layers "F.Cu" "B.Cu") (free) (net 0))
+  (via (at 138.1 125.4) (size 4) (drill 2.6) (layers "F.Cu" "B.Cu") (free) (net 0))
+  (via (at 61.9 74.6) (size 4) (drill 2.6) (layers "F.Cu" "B.Cu") (free) (net 0))
   (segment (start 93.52 77.45) (end 93.52 79.042) (width 0.25) (layer "F.Cu") (net 1))
   (segment (start 97.293554 99.06) (end 97.79 99.06) (width 0.25) (layer "F.Cu") (net 1))
